File: Differential Probe.kicad_pcb (KiCad board)
At the start: 4 copper layers, 2 x 18 mm, 105 parts, among them J1 Conn_Coaxial, J2 Conn_Coaxial, J3 USB_C_Receptacle_PowerOnly_6P, J4 Conn_Coaxial, SW1 SW_SP3T_NINGI, U1 BQ24072RGT, U2 OPA810xD, U3 OPA810xD, U4 OPA810xD, U5 TPS65135RTER

Commit message: PCB layout 90%
Parts:
- removed C1, C2, C3, C4: 10p, Capacitor_SMD:C_1206_3216Metric_Pad1.33x1.80mm_HandSolder
- removed SW1: SW_SP3T_NINGI, Library:SR17A1320F39N
- added C46: 10p, Capacitor_SMD:C_1206_3216Metric_Pad1.33x1.80mm_HandSolder, F.Cu at (85.5, 102.5)
- added C47: 10p, Capacitor_SMD:C_1206_3216Metric_Pad1.33x1.80mm_HandSolder, F.Cu at (85.5, 108.0)
- added C48: 10p, Capacitor_SMD:C_1206_3216Metric_Pad1.33x1.80mm_HandSolder, F.Cu at (85.5, 124.9)
- added C49: 10p, Capacitor_SMD:C_1206_3216Metric_Pad1.33x1.80mm_HandSolder, F.Cu at (85.5, 130.4)
- added C50: 4u7, Capacitor_SMD:C_0603_1608Metric_Pad1.08x0.95mm_HandSolder, B.Cu at (141.0, 134.9)
- added C51: 4u7, Capacitor_SMD:C_0603_1608Metric_Pad1.08x0.95mm_HandSolder, B.Cu at (141.0, 141.7)
- added H1: MountingHole_Pad, MountingHole:MountingHole_3.2mm_M3_DIN965_Pad, F.Cu at (85.5, 116.5)
- added H2: MountingHole_Pad, MountingHole:MountingHole_3.2mm_M3_DIN965_Pad, F.Cu at (118.5, 96.5)
- added H3: MountingHole_Pad, MountingHole:MountingHole_3.2mm_M3_DIN965_Pad, F.Cu at (184.5, 96.5)
- added H4: MountingHole_Pad, MountingHole:MountingHole_3.2mm_M3_DIN965_Pad, F.Cu at (184.5, 146.5)
- added H5: MountingHole_Pad, MountingHole:MountingHole_3.2mm_M3_DIN965_Pad, F.Cu at (97.5, 146.5)
- added R42: 200, Resistor_SMD:R_0603_1608Metric_Pad0.98x0.95mm_HandSolder, F.Cu at (146.8, 125.6)
- added SW2: SW_DIP_x03, Button_Switch_SMD:SW_DIP_SPSTx03_Slide_KingTek_DSHP03TS_W7.62mm_P1.27mm, F.Cu at (144.2, 116.4)
- BT1, C31, C38, C39, C44, C45, L1, R35, R36, R37, R38, R39, R40, R41, U5: moved to B.Cu
- C20, C29, C30: footprint Capacitor_SMD:C_0805_2012Metric_Pad1.18x1.45mm_HandSolder -> Capacitor_SMD:C_0603_1608Metric_Pad1.08x0.95mm_HandSolder
- C32, C33, C34, C35: footprint Capacitor_SMD:C_1206_3216Metric_Pad1.33x1.80mm_HandSolder -> Capacitor_SMD:C_0603_1608Metric_Pad1.08x0.95mm_HandSolder; moved to B.Cu
- C36, C37, C40, C41, C42, C43: footprint Capacitor_SMD:C_1206_3216Metric_Pad1.33x1.80mm_HandSolder -> Capacitor_SMD:C_0603_1608Metric_Pad1.08x0.95mm_HandSolder
- J1, J2: value Conn_Coaxial -> Conn_01x01_Pin; footprint Connector_Coaxial:BNC_Amphenol_B6252HB-NPP3G-50_Horizontal -> NetTie:NetTie-2_SMD_Pad2.0mm
- moved BT1 112.3 mm to (105.4, 140.2)
- moved R18 108.0 mm to (151.5, 147.2)
- moved C44 107.4 mm to (120.8, 136.1), turned to -90 degrees
- moved R24 106.1 mm to (151.5, 142.4)
- moved R21 106.1 mm to (153.6, 138.8)
- moved R17 106.0 mm to (155.5, 138.8)
- moved R19 105.9 mm to (157.4, 138.8)
- moved C20 105.8 mm to (159.3, 138.8)
- moved C17 105.5 mm to (164.0, 135.0), turned to -90 degrees
- moved R20 105.4 mm to (162.3, 141.2)
- moved U1 105.4 mm to (156.5, 144.4)
- moved R40 105.3 mm to (124.6, 134.6), turned to 0 degrees
- moved R26 105.3 mm to (162.3, 143.0)
- moved D4 105.1 mm to (162.3, 144.8)
- moved D3 105.0 mm to (162.3, 146.6)
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Connections:
- C18 pad 2: GNDA -> GND
- C19 pad 1: GNDA -> GND
- C21 pad 2: GNDA -> GND
- C22 pad 1: GNDA -> GND
- C23 pad 2: GNDA -> GND
- C24 pad 1: GNDA -> GND
- C25 pad 2: GNDA -> GND
- C26 pad 1: GNDA -> GND
- C36 pad 2: Net-(C36-Pad2) -> GND
- C37 pad 1: Net-(C36-Pad2) -> GND
- C40 pad 2: Net-(C36-Pad2) -> GND
- C41 pad 1: Net-(C36-Pad2) -> GND
- C42 pad 2: Net-(C36-Pad2) -> GND
- C43 pad 1: Net-(C36-Pad2) -> GND
- J1 pad 2: GNDA -> (no net)
- J2 pad 2: GNDA -> (no net)
- J4 pad 2: GNDA -> GND
- R31 pad 2: GNDA -> GND
- RV1 pad 2: GNDA -> GND
Routing:
- net GND: track 0.00 -> 128.3 mm, vias 0 -> 103
- net Net-(BT1-+): track 0.00 -> 55.9 mm
- net Net-(D2B-K1A2): track 0.00 -> 54.9 mm
- net Net-(D2A-K3A4): track 0.00 -> 51.1 mm
- net Net-(C28-Pad2): track 0.00 -> 26.1 mm
- net +6V: track 0.00 -> 23.0 mm, vias 0 -> 5
- net Net-(C27-Pad1): track 0.00 -> 20.9 mm
- net -6V: track 0.00 -> 20.0 mm, vias 0 -> 7
- net Net-(R32-Pad2): track 0.00 -> 17.7 mm
- net OUT: track 0.00 -> 14.2 mm, vias 0 -> 8
- net Net-(C13-Pad1): track 0.00 -> 13.5 mm
- net Net-(C8-Pad2): track 0.00 -> 13.4 mm
- net Net-(C12-Pad1): track 0.00 -> 13.4 mm
- net Net-(C13-Pad2): track 0.00 -> 13.3 mm
- net Net-(C10-Pad1): track 0.00 -> 13.3 mm
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- added copper zone on B.Cu, net GND
- added copper zone on F.Cu, net GND
- added copper zone on In1.Cu, net GND
- added copper zone on In2.Cu, net GND
- added copper zone on F.Cu, net Net-(C11-Pad1)
- added copper zone on B.Cu, net Net-(C34-Pad1)
- added copper zone on B.Cu, net Net-(C35-Pad2)
- added copper zone on F.Cu, net Net-(F1-Pad1)
- added copper zone on B.Cu, net Net-(L1-Pad1)
- added copper zone on B.Cu, net Net-(L1-Pad2)
- added copper zone on F.Cu, net Net-(U1-IN)
- added copper zone on B.Cu, net OUT
- added copper zone on F.Cu, net OUT
Other:
- board size 2 x 18 mm -> 115.5 x 60 mm

Commit message: Ready to check
Parts:
- moved J4 1.41 mm to (175.4, 116.5)
- moved H3 0.50 mm to (184.0, 96.5)
- moved H4 0.50 mm to (184.0, 146.5)
- moved J3 0.48 mm to (185.6, 136.0)
- moved R33 0.30 mm to (170.2, 115.5)
- moved R34 0.30 mm to (170.2, 118.5)
- moved C30 0.20 mm to (156.5, 147.8)
Connections:
- C47 pad 2: GND -> Earth
- C48 pad 1: GND -> Earth
- H1 pad 1: GND -> Earth
Routing:
- net -6V: track 20.0 -> 56.0 mm, vias 7 -> 13
- net GND: track 128.3 -> 110.5 mm, vias 103 -> 113
- net +6V: track 23.0 -> 38.5 mm
- net Earth: track 0.00 -> 13.8 mm
- net Net-(C5-Pad1): track 13.3 -> 10.1 mm
- net Net-(C8-Pad2): track 13.4 -> 10.2 mm
- net Net-(C6-Pad2): track 13.3 -> 10.1 mm
- net Net-(C13-Pad2): track 13.3 -> 10.1 mm
- net Net-(C13-Pad1): track 13.5 -> 10.3 mm
- net Net-(C12-Pad1): track 13.4 -> 10.2 mm
- net Net-(C10-Pad2): track 13.3 -> 10.1 mm
- net Net-(C10-Pad1): track 13.3 -> 10.1 mm
- net Net-(D2A-K3A4): track 51.1 -> 49.2 mm
- net Net-(J2-Pin_1): track 13.0 -> 11.4 mm
- net Net-(J1-Pin_1): track 13.1 -> 11.5 mm
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- added copper zone on B.Cu, net +6V
- added copper zone on B.Cu, net -6V
- added copper zone on F.Cu, net -6V
- added copper zone on B.Cu, net Earth
- added copper zone on F.Cu, net Earth
- removed copper zone on F.Cu, net GND
Other:
- board size 115.5 x 60 mm -> 115 x 60 mm
- board text added: "0 3 2 1"
- board text added: "0V to +/- 1500V"
- board text added: "1"
- board text added: "2025 POLAND"
- board text added: "3"
- board text added: "750 7.5 75 350"
- board text added: "CMRR"
- board text added: "Chassis"
- board text added: "DIFF PROBE rev 1.0"
- board text added: "Designed by Michal Karas"
- board text added: "GAIN"
- board text added: "NEG"
- board text added: "OUTPUT"
- board text added: "PCB3D_BR_Differential Probe"
- board text added: "PCB3D_TL_Differential Probe"
- board text added: "POS"
- board text added: "SHUNT(Only One)"
- board text added: "and Aleksander Kaweczyński"
